Commit message: updated camera.xacro

File: models/camera.xacro (robot description, xacro)
@@ -26,5 +26,5 @@
   </link>
   <joint name="${uav_name}_camera_joint" type="fixed">
-    <parent link="$(arg parent_link)"/>
+    <parent link="${parent_link}"/>
     <child link="${uav_name}_camera_link"/>
     <origin xyz="0 0 0.1" rpy="0 0 0"/> <!-- Mounted 10cm above base_link -->
@@ -51,5 +51,5 @@
         <always_on>true</always_on>
         <update_rate>30.0</update_rate>
-        <camera_name>$(arg uav_name)/camera</camera_name>
+        <camera_name>${uav_name}/camera</camera_name>
         <image_topic_name>image_raw</image_topic_name>
         <camera_info_topic_name>camera_info</camera_info_topic_name>

Commit message: updated camera xacro

File: models/camera.xacro (robot description, xacro)
@@ -1,60 +1,60 @@
 <?xml version="1.0"?>
-<robot xmlns:xacro="http://ros.org/wiki/xacro" name="camera_${uav_name}">
-  <xacro:arg name="uav_name" default="uav0"/>
-  <xacro:arg name="parent_link" default="base_link"/>
-  <link name="${uav_name}_camera_link">
-    <inertial>
-      <mass value="0.1"/>
-      <origin xyz="0 0 0"/>
-      <inertia ixx="0.0001" ixy="0.0" ixz="0.0" iyy="0.0001" iyz="0.0" izz="0.0001"/>
-    </inertial>
-    <visual>
-      <origin xyz="0 0 0" rpy="0 0 0"/>
-      <geometry>
-        <box size="0.05 0.05 0.02"/>
-      </geometry>
-      <material name="gray">
-        <color rgba="0.5 0.5 0.5 1.0"/>
-      </material>
-    </visual>
-    <collision>
-      <origin xyz="0 0 0" rpy="0 0 0"/>
-      <geometry>
-        <box size="0.05 0.05 0.02"/>
-      </geometry>
-    </collision>
-  </link>
-  <joint name="${uav_name}_camera_joint" type="fixed">
-    <parent link="${parent_link}"/>
-    <child link="${uav_name}_camera_link"/>
-    <origin xyz="0 0 0.1" rpy="0 0 0"/> <!-- Mounted 10cm above base_link -->
-  </joint>
-  <gazebo reference="${uav_name}_camera_link">
-    <sensor type="camera" name="${uav_name}_camera_sensor">
-      <pose>0 0 0 0 0 0</pose>
-      <camera>
-        <horizontal_fov>1.3962634</horizontal_fov>
-        <image>
-          <width>640</width>
-          <height>480</height>
-          <format>R8G8B8</format>
-        </image>
-        <clip>
-          <near>0.05</near>
-          <far>100.0</far>
-        </clip>
-      </camera>
-      <always_on>true</always_on>
-      <update_rate>30.0</update_rate>
-      <visualize>true</visualize>
-      <plugin name="${uav_name}_camera_controller" filename="libgazebo_ros_camera.so">
+<xacro:macro name="camera" params="uav_name parent_link">
+  <robot xmlns:xacro="http://ros.org/wiki/xacro" name="camera_${uav_name}">
+    <link name="${uav_name}_camera_link">
+      <inertial>
+        <mass value="0.1"/>
+        <origin xyz="0 0 0"/>
+        <inertia ixx="0.0001" ixy="0.0" ixz="0.0" iyy="0.0001" iyz="0.0" izz="0.0001"/>
+      </inertial>
+      <visual>
+        <origin xyz="0 0 0" rpy="0 0 0"/>
+        <geometry>
+          <box size="0.05 0.05 0.02"/>
+        </geometry>
+        <material name="gray">
+          <color rgba="0.5 0.5 0.5 1.0"/>
+        </material>
+      </visual>
+      <collision>
+        <origin xyz="0 0 0" rpy="0 0 0"/>
+        <geometry>
+          <box size="0.05 0.05 0.02"/>
+        </geometry>
+      </collision>
+    </link>
+    <joint name="${uav_name}_camera_joint" type="fixed">
+      <parent link="${parent_link}"/>
+      <child link="${uav_name}_camera_link"/>
+      <origin xyz="0 0 0.1" rpy="0 0 0"/>
+    </joint>
+    <gazebo reference="${uav_name}_camera_link">
+      <sensor type="camera" name="${uav_name}_camera_sensor">
+        <pose>0 0 0 0 0 0</pose>
+        <camera>
+          <horizontal_fov>1.3962634</horizontal_fov>
+          <image>
+            <width>640</width>
+            <height>480</height>
+            <format>R8G8B8</format>
+          </image>
+          <clip>
+            <near>0.05</near>
+            <far>100.0</far>
+          </clip>
+        </camera>
         <always_on>true</always_on>
         <update_rate>30.0</update_rate>
-        <camera_name>${uav_name}/camera</camera_name>
-        <image_topic_name>image_raw</image_topic_name>
-        <camera_info_topic_name>camera_info</camera_info_topic_name>
-        <frame_name>${uav_name}_camera_link</frame_name>
-      </plugin>
-    </sensor>
-  </gazebo>
-</robot>
+        <visualize>true</visualize>
+        <plugin name="${uav_name}_camera_controller" filename="libgazebo_ros_camera.so">
+          <always_on>true</always_on>
+          <update_rate>30.0</update_rate>
+          <camera_name>${uav_name}/camera</camera_name>
+          <image_topic_name>image_raw</image_topic_name>
+          <camera_info_topic_name>camera_info</camera_info_topic_name>
+          <frame_name>${uav_name}_camera_link</frame_name>
+        </plugin>
+      </sensor>
+    </gazebo>
+  </robot>
+</xacro:macro>

Commit message: Update camera.xacro

File: models/camera.xacro (robot description, xacro)
@@ -1,60 +1,64 @@
 <?xml version="1.0"?>
-<xacro:macro name="camera" params="uav_name parent_link">
-  <robot xmlns:xacro="http://ros.org/wiki/xacro" name="camera_${uav_name}">
-    <link name="${uav_name}_camera_link">
-      <inertial>
-        <mass value="0.1"/>
-        <origin xyz="0 0 0"/>
-        <inertia ixx="0.0001" ixy="0.0" ixz="0.0" iyy="0.0001" iyz="0.0" izz="0.0001"/>
-      </inertial>
-      <visual>
-        <origin xyz="0 0 0" rpy="0 0 0"/>
-        <geometry>
-          <box size="0.05 0.05 0.02"/>
-        </geometry>
-        <material name="gray">
-          <color rgba="0.5 0.5 0.5 1.0"/>
-        </material>
-      </visual>
-      <collision>
-        <origin xyz="0 0 0" rpy="0 0 0"/>
-        <geometry>
-          <box size="0.05 0.05 0.02"/>
-        </geometry>
-      </collision>
-    </link>
-    <joint name="${uav_name}_camera_joint" type="fixed">
-      <parent link="${parent_link}"/>
-      <child link="${uav_name}_camera_link"/>
-      <origin xyz="0 0 0.1" rpy="0 0 0"/>
-    </joint>
-    <gazebo reference="${uav_name}_camera_link">
-      <sensor type="camera" name="${uav_name}_camera_sensor">
-        <pose>0 0 0 0 0 0</pose>
-        <camera>
-          <horizontal_fov>1.3962634</horizontal_fov>
-          <image>
-            <width>640</width>
-            <height>480</height>
-            <format>R8G8B8</format>
-          </image>
-          <clip>
-            <near>0.05</near>
-            <far>100.0</far>
-          </clip>
-        </camera>
+<robot xmlns:xacro="http://www.ros.org/wiki/xacro" name="camera_${uav_name}">
+  <!-- Arguments -->
+  <xacro:arg name="uav_name" default="uav0"/>
+  <xacro:arg name="parent_link" default="base_link"/>
+  <!-- Camera link -->
+  <link name="${uav_name}_camera_link">
+    <inertial>
+      <mass value="0.1"/>
+      <origin xyz="0 0 0"/>
+      <inertia ixx="0.0001" ixy="0.0" ixz="0.0" iyy="0.0001" iyz="0.0" izz="0.0001"/>
+    </inertial>
+    <visual>
+      <origin xyz="0 0 0" rpy="0 0 0"/>
+      <geometry>
+        <box size="0.05 0.05 0.02"/>
+      </geometry>
+      <material name="gray">
+        <color rgba="0.5 0.5 0.5 1.0"/>
+      </material>
+    </visual>
+    <collision>
+      <origin xyz="0 0 0" rpy="0 0 0"/>
+      <geometry>
+        <box size="0.05 0.05 0.02"/>
+      </geometry>
+    </collision>
+  </link>
+  <!-- Camera joint -->
+  <joint name="${uav_name}_camera_joint" type="fixed">
+    <parent link="${parent_link}"/>
+    <child link="${uav_name}_camera_link"/>
+    <origin xyz="0 0 0.1" rpy="0 0 0"/> <!-- Mounted 10cm above base_link -->
+  </joint>
+  <!-- Gazebo sensor plugin -->
+  <gazebo reference="${uav_name}_camera_link">
+    <sensor type="camera" name="${uav_name}_camera_sensor">
+      <pose>0 0 0 0 0 0</pose>
+      <camera>
+        <horizontal_fov>1.3962634</horizontal_fov>
+        <image>
+          <width>640</width>
+          <height>480</height>
+          <format>R8G8B8</format>
+        </image>
+        <clip>
+          <near>0.05</near>
+          <far>100.0</far>
+        </clip>
+      </camera>
+      <always_on>true</always_on>
+      <update_rate>30.0</update_rate>
+      <visualize>true</visualize>
+      <plugin name="${uav_name}_camera_controller" filename="libgazebo_ros_camera.so">
         <always_on>true</always_on>
         <update_rate>30.0</update_rate>
-        <visualize>true</visualize>
-        <plugin name="${uav_name}_camera_controller" filename="libgazebo_ros_camera.so">
-          <always_on>true</always_on>
-          <update_rate>30.0</update_rate>
-          <camera_name>${uav_name}/camera</camera_name>
-          <image_topic_name>image_raw</image_topic_name>
-          <camera_info_topic_name>camera_info</camera_info_topic_name>
-          <frame_name>${uav_name}_camera_link</frame_name>
-        </plugin>
-      </sensor>
-    </gazebo>
-  </robot>
-</xacro:macro>
+        <camera_name>${uav_name}/camera</camera_name>
+        <image_topic_name>image_raw</image_topic_name>
+        <camera_info_topic_name>camera_info</camera_info_topic_name>
+        <frame_name>${uav_name}_camera_link</frame_name>
+      </plugin>
+    </sensor>
+  </gazebo>
+</robot>

Commit message: Update camera.xacro

File: models/camera.xacro (robot description, xacro)
@@ -1,65 +1,67 @@
 <?xml version="1.0"?>
 <robot xmlns:xacro="http://www.ros.org/wiki/xacro">
-  <!-- Define arguments -->
+  <!-- Argument definitions -->
   <xacro:arg name="uav_name" default="uav0"/>
   <xacro:arg name="parent_link" default="base_link"/>
+  <!-- Robot definition -->
   <robot name="camera_${uav_name}">
-  <!-- Camera link -->
-  <link name="${uav_name}_camera_link">
-    <inertial>
-      <mass value="0.1"/>
-      <origin xyz="0 0 0"/>
-      <inertia ixx="0.0001" ixy="0.0" ixz="0.0" iyy="0.0001" iyz="0.0" izz="0.0001"/>
-    </inertial>
-    <visual>
-      <origin xyz="0 0 0" rpy="0 0 0"/>
-      <geometry>
-        <box size="0.05 0.05 0.02"/>
-      </geometry>
-      <material name="gray">
-        <color rgba="0.5 0.5 0.5 1.0"/>
-      </material>
-    </visual>
-    <collision>
-      <origin xyz="0 0 0" rpy="0 0 0"/>
-      <geometry>
-        <box size="0.05 0.05 0.02"/>
-      </geometry>
-    </collision>
-  </link>
-  <!-- Camera joint -->
-  <joint name="${uav_name}_camera_joint" type="fixed">
-    <parent link="${parent_link}"/>
-    <child link="${uav_name}_camera_link"/>
-    <origin xyz="0 0 0.1" rpy="0 0 0"/> <!-- Mounted 10cm above base_link -->
-  </joint>
-  <!-- Gazebo sensor plugin -->
-  <gazebo reference="${uav_name}_camera_link">
-    <sensor type="camera" name="${uav_name}_camera_sensor">
-      <pose>0 0 0 0 0 0</pose>
-      <camera>
-        <horizontal_fov>1.3962634</horizontal_fov>
-        <image>
-          <width>640</width>
-          <height>480</height>
-          <format>R8G8B8</format>
-        </image>
-        <clip>
-          <near>0.05</near>
-          <far>100.0</far>
-        </clip>
-      </camera>
-      <always_on>true</always_on>
-      <update_rate>30.0</update_rate>
-      <visualize>true</visualize>
-      <plugin name="${uav_name}_camera_controller" filename="libgazebo_ros_camera.so">
+    <!-- Define links, joints, and other properties here -->
+    <link name="${uav_name}_camera_link">
+      <inertial>
+        <mass value="0.1"/>
+        <origin xyz="0 0 0"/>
+        <inertia ixx="0.0001" ixy="0.0" ixz="0.0" iyy="0.0001" iyz="0.0" izz="0.0001"/>
+      </inertial>
+      <visual>
+        <origin xyz="0 0 0" rpy="0 0 0"/>
+        <geometry>
+          <box size="0.05 0.05 0.02"/>
+        </geometry>
+        <material name="gray">
+          <color rgba="0.5 0.5 0.5 1.0"/>
+        </material>
+      </visual>
+      <collision>
+        <origin xyz="0 0 0" rpy="0 0 0"/>
+        <geometry>
+          <box size="0.05 0.05 0.02"/>
+        </geometry>
+      </collision>
+    </link>
+    <!-- Joint definition -->
+    <joint name="${uav_name}_camera_joint" type="fixed">
+      <parent link="${parent_link}"/>
+      <child link="${uav_name}_camera_link"/>
+      <origin xyz="0 0 0.1" rpy="0 0 0"/> <!-- Mounted 10cm above base_link -->
+    </joint>
+    <!-- Gazebo sensor plugin -->
+    <gazebo reference="${uav_name}_camera_link">
+      <sensor type="camera" name="${uav_name}_camera_sensor">
+        <pose>0 0 0 0 0 0</pose>
+        <camera>
+          <horizontal_fov>1.3962634</horizontal_fov>
+          <image>
+            <width>640</width>
+            <height>480</height>
+            <format>R8G8B8</format>
+          </image>
+          <clip>
+            <near>0.05</near>
+            <far>100.0</far>
+          </clip>
+        </camera>
         <always_on>true</always_on>
         <update_rate>30.0</update_rate>
-        <camera_name>${uav_name}/camera</camera_name>
-        <image_topic_name>image_raw</image_topic_name>
-        <camera_info_topic_name>camera_info</camera_info_topic_name>
-        <frame_name>${uav_name}_camera_link</frame_name>
-      </plugin>
-    </sensor>
-  </gazebo>
+        <visualize>true</visualize>
+        <plugin name="${uav_name}_camera_controller" filename="libgazebo_ros_camera.so">
+          <always_on>true</always_on>
+          <update_rate>30.0</update_rate>
+          <camera_name>${uav_name}/camera</camera_name>
+          <image_topic_name>image_raw</image_topic_name>
+          <camera_info_topic_name>camera_info</camera_info_topic_name>
+          <frame_name>${uav_name}_camera_link</frame_name>
+        </plugin>
+      </sensor>
+    </gazebo>
+  </robot>
 </robot>

Commit message: Update camera.xacro

File: models/camera.xacro (robot description, xacro)
@@ -1,67 +1,64 @@
 <?xml version="1.0"?>
 <robot xmlns:xacro="http://www.ros.org/wiki/xacro">
-  <!-- Argument definitions -->
+  <!-- Define arguments -->
   <xacro:arg name="uav_name" default="uav0"/>
   <xacro:arg name="parent_link" default="base_link"/>
-  <!-- Robot definition -->
-  <robot name="camera_${uav_name}">
-    <!-- Define links, joints, and other properties here -->
-    <link name="${uav_name}_camera_link">
-      <inertial>
-        <mass value="0.1"/>
-        <origin xyz="0 0 0"/>
-        <inertia ixx="0.0001" ixy="0.0" ixz="0.0" iyy="0.0001" iyz="0.0" izz="0.0001"/>
-      </inertial>
-      <visual>
-        <origin xyz="0 0 0" rpy="0 0 0"/>
-        <geometry>
-          <box size="0.05 0.05 0.02"/>
-        </geometry>
-        <material name="gray">
-          <color rgba="0.5 0.5 0.5 1.0"/>
-        </material>
-      </visual>
-      <collision>
-        <origin xyz="0 0 0" rpy="0 0 0"/>
-        <geometry>
-          <box size="0.05 0.05 0.02"/>
-        </geometry>
-      </collision>
-    </link>
-    <!-- Joint definition -->
-    <joint name="${uav_name}_camera_joint" type="fixed">
-      <parent link="${parent_link}"/>
-      <child link="${uav_name}_camera_link"/>
-      <origin xyz="0 0 0.1" rpy="0 0 0"/> <!-- Mounted 10cm above base_link -->
-    </joint>
-    <!-- Gazebo sensor plugin -->
-    <gazebo reference="${uav_name}_camera_link">
-      <sensor type="camera" name="${uav_name}_camera_sensor">
-        <pose>0 0 0 0 0 0</pose>
-        <camera>
-          <horizontal_fov>1.3962634</horizontal_fov>
-          <image>
-            <width>640</width>
-            <height>480</height>
-            <format>R8G8B8</format>
-          </image>
-          <clip>
-            <near>0.05</near>
-            <far>100.0</far>
-          </clip>
-        </camera>
+  <!-- Define the camera link -->
+  <link name="${uav_name}_camera_link">
+    <inertial>
+      <mass value="0.1"/>
+      <origin xyz="0 0 0"/>
+      <inertia ixx="0.0001" ixy="0.0" ixz="0.0" iyy="0.0001" iyz="0.0" izz="0.0001"/>
+    </inertial>
+    <visual>
+      <origin xyz="0 0 0" rpy="0 0 0"/>
+      <geometry>
+        <box size="0.05 0.05 0.02"/>
+      </geometry>
+      <material name="gray">
+        <color rgba="0.5 0.5 0.5 1.0"/>
+      </material>
+    </visual>
+    <collision>
+      <origin xyz="0 0 0" rpy="0 0 0"/>
+      <geometry>
+        <box size="0.05 0.05 0.02"/>
+      </geometry>
+    </collision>
+  </link>
+  <!-- Define the joint -->
+  <joint name="${uav_name}_camera_joint" type="fixed">
+    <parent link="${parent_link}"/>
+    <child link="${uav_name}_camera_link"/>
+    <origin xyz="0 0 0.1" rpy="0 0 0"/> <!-- Mounted 10cm above base_link -->
+  </joint>
+  <!-- Gazebo camera sensor plugin -->
+  <gazebo reference="${uav_name}_camera_link">
+    <sensor type="camera" name="${uav_name}_camera_sensor">
+      <pose>0 0 0 0 0 0</pose>
+      <camera>
+        <horizontal_fov>1.3962634</horizontal_fov>
+        <image>
+          <width>640</width>
+          <height>480</height>
+          <format>R8G8B8</format>
+        </image>
+        <clip>
+          <near>0.05</near>
+          <far>100.0</far>
+        </clip>
+      </camera>
+      <always_on>true</always_on>
+      <update_rate>30.0</update_rate>
+      <visualize>true</visualize>
+      <plugin name="${uav_name}_camera_controller" filename="libgazebo_ros_camera.so">
         <always_on>true</always_on>
         <update_rate>30.0</update_rate>
-        <visualize>true</visualize>
-        <plugin name="${uav_name}_camera_controller" filename="libgazebo_ros_camera.so">
-          <always_on>true</always_on>
-          <update_rate>30.0</update_rate>
-          <camera_name>${uav_name}/camera</camera_name>
-          <image_topic_name>image_raw</image_topic_name>
-          <camera_info_topic_name>camera_info</camera_info_topic_name>
-          <frame_name>${uav_name}_camera_link</frame_name>
-        </plugin>
-      </sensor>
-    </gazebo>
-  </robot>
+        <camera_name>${uav_name}/camera</camera_name>
+        <image_topic_name>image_raw</image_topic_name>
+        <camera_info_topic_name>camera_info</camera_info_topic_name>
+        <frame_name>${uav_name}_camera_link</frame_name>
+      </plugin>
+    </sensor>
+  </gazebo>
 </robot>

Commit message: Update camera.xacro

File: models/camera.xacro (robot description, xacro)
@@ -1,64 +1,64 @@
 <?xml version="1.0"?>
 <robot xmlns:xacro="http://www.ros.org/wiki/xacro">
-  <!-- Define arguments -->
+  <!-- Argument definitions must come first -->
   <xacro:arg name="uav_name" default="uav0"/>
   <xacro:arg name="parent_link" default="base_link"/>
-  <!-- Define the camera link -->
-  <link name="${uav_name}_camera_link">
-    <inertial>
-      <mass value="0.1"/>
-      <origin xyz="0 0 0"/>
-      <inertia ixx="0.0001" ixy="0.0" ixz="0.0" iyy="0.0001" iyz="0.0" izz="0.0001"/>
-    </inertial>
-    <visual>
-      <origin xyz="0 0 0" rpy="0 0 0"/>
-      <geometry>
-        <box size="0.05 0.05 0.02"/>
-      </geometry>
-      <material name="gray">
-        <color rgba="0.5 0.5 0.5 1.0"/>
-      </material>
-    </visual>
-    <collision>
-      <origin xyz="0 0 0" rpy="0 0 0"/>
-      <geometry>
-        <box size="0.05 0.05 0.02"/>
-      </geometry>
-    </collision>
-  </link>
-  <!-- Define the joint -->
-  <joint name="${uav_name}_camera_joint" type="fixed">
-    <parent link="${parent_link}"/>
-    <child link="${uav_name}_camera_link"/>
-    <origin xyz="0 0 0.1" rpy="0 0 0"/> <!-- Mounted 10cm above base_link -->
-  </joint>
-  <!-- Gazebo camera sensor plugin -->
-  <gazebo reference="${uav_name}_camera_link">
-    <sensor type="camera" name="${uav_name}_camera_sensor">
-      <pose>0 0 0 0 0 0</pose>
-      <camera>
-        <horizontal_fov>1.3962634</horizontal_fov>
-        <image>
-          <width>640</width>
-          <height>480</height>
-          <format>R8G8B8</format>
-        </image>
-        <clip>
-          <near>0.05</near>
-          <far>100.0</far>
-        </clip>
-      </camera>
-      <always_on>true</always_on>
-      <update_rate>30.0</update_rate>
-      <visualize>true</visualize>
-      <plugin name="${uav_name}_camera_controller" filename="libgazebo_ros_camera.so">
+  <!-- Now you can use the uav_name variable here -->
+  <robot name="camera_${uav_name}">
+    <link name="${uav_name}_camera_link">
+      <inertial>
+        <mass value="0.1"/>
+        <origin xyz="0 0 0"/>
+        <inertia ixx="0.0001" ixy="0.0" ixz="0.0" iyy="0.0001" iyz="0.0" izz="0.0001"/>
+      </inertial>
+      <visual>
+        <origin xyz="0 0 0" rpy="0 0 0"/>
+        <geometry>
+          <box size="0.05 0.05 0.02"/>
+        </geometry>
+        <material name="gray">
+          <color rgba="0.5 0.5 0.5 1.0"/>
+        </material>
+      </visual>
+      <collision>
+        <origin xyz="0 0 0" rpy="0 0 0"/>
+        <geometry>
+          <box size="0.05 0.05 0.02"/>
+        </geometry>
+      </collision>
+    </link>
+    <joint name="${uav_name}_camera_joint" type="fixed">
+      <parent link="${parent_link}"/>
+      <child link="${uav_name}_camera_link"/>
+      <origin xyz="0 0 0.1" rpy="0 0 0"/> <!-- Mounted 10cm above base_link -->
+    </joint>
+    <gazebo reference="${uav_name}_camera_link">
+      <sensor type="camera" name="${uav_name}_camera_sensor">
+        <pose>0 0 0 0 0 0</pose>
+        <camera>
+          <horizontal_fov>1.3962634</horizontal_fov>
+          <image>
+            <width>640</width>
+            <height>480</height>
+            <format>R8G8B8</format>
+          </image>
+          <clip>
+            <near>0.05</near>
+            <far>100.0</far>
+          </clip>
+        </camera>
         <always_on>true</always_on>
         <update_rate>30.0</update_rate>
-        <camera_name>${uav_name}/camera</camera_name>
-        <image_topic_name>image_raw</image_topic_name>
-        <camera_info_topic_name>camera_info</camera_info_topic_name>
-        <frame_name>${uav_name}_camera_link</frame_name>
-      </plugin>
-    </sensor>
-  </gazebo>
+        <visualize>true</visualize>
+        <plugin name="${uav_name}_camera_controller" filename="libgazebo_ros_camera.so">
+          <always_on>true</always_on>
+          <update_rate>30.0</update_rate>
+          <camera_name>${uav_name}/camera</camera_name>
+          <image_topic_name>image_raw</image_topic_name>
+          <camera_info_topic_name>camera_info</camera_info_topic_name>
+          <frame_name>${uav_name}_camera_link</frame_name>
+        </plugin>
+      </sensor>
+    </gazebo>
+  </robot>
 </robot>
