Commit message: Update camera.xacro

File: models/camera.xacro (robot description, xacro)
@@ -1,64 +1,64 @@
 <?xml version="1.0"?>
 <robot xmlns:xacro="http://www.ros.org/wiki/xacro">
-  <!-- Argument definitions must come first -->
+  <!-- Define arguments -->
   <xacro:arg name="uav_name" default="uav0"/>
   <xacro:arg name="parent_link" default="base_link"/>
-  <!-- Now you can use the uav_name variable here -->
-  <robot name="camera_${uav_name}">
-    <link name="${uav_name}_camera_link">
-      <inertial>
-        <mass value="0.1"/>
-        <origin xyz="0 0 0"/>
-        <inertia ixx="0.0001" ixy="0.0" ixz="0.0" iyy="0.0001" iyz="0.0" izz="0.0001"/>
-      </inertial>
-      <visual>
-        <origin xyz="0 0 0" rpy="0 0 0"/>
-        <geometry>
-          <box size="0.05 0.05 0.02"/>
-        </geometry>
-        <material name="gray">
-          <color rgba="0.5 0.5 0.5 1.0"/>
-        </material>
-      </visual>
-      <collision>
-        <origin xyz="0 0 0" rpy="0 0 0"/>
-        <geometry>
-          <box size="0.05 0.05 0.02"/>
-        </geometry>
-      </collision>
-    </link>
-    <joint name="${uav_name}_camera_joint" type="fixed">
-      <parent link="${parent_link}"/>
-      <child link="${uav_name}_camera_link"/>
-      <origin xyz="0 0 0.1" rpy="0 0 0"/> <!-- Mounted 10cm above base_link -->
-    </joint>
-    <gazebo reference="${uav_name}_camera_link">
-      <sensor type="camera" name="${uav_name}_camera_sensor">
-        <pose>0 0 0 0 0 0</pose>
-        <camera>
-          <horizontal_fov>1.3962634</horizontal_fov>
-          <image>
-            <width>640</width>
-            <height>480</height>
-            <format>R8G8B8</format>
-          </image>
-          <clip>
-            <near>0.05</near>
-            <far>100.0</far>
-          </clip>
-        </camera>
+  <!-- Define the camera link -->
+  <link name="$(arg uav_name)_camera_link">
+    <inertial>
+      <mass value="0.1"/>
+      <origin xyz="0 0 0"/>
+      <inertia ixx="0.0001" ixy="0.0" ixz="0.0" iyy="0.0001" iyz="0.0" izz="0.0001"/>
+    </inertial>
+    <visual>
+      <origin xyz="0 0 0" rpy="0 0 0"/>
+      <geometry>
+        <box size="0.05 0.05 0.02"/>
+      </geometry>
+      <material name="gray">
+        <color rgba="0.5 0.5 0.5 1.0"/>
+      </material>
+    </visual>
+    <collision>
+      <origin xyz="0 0 0" rpy="0 0 0"/>
+      <geometry>
+        <box size="0.05 0.05 0.02"/>
+      </geometry>
+    </collision>
+  </link>
+  <!-- Define the joint -->
+  <joint name="$(arg uav_name)_camera_joint" type="fixed">
+    <parent link="$(arg parent_link)"/>
+    <child link="$(arg uav_name)_camera_link"/>
+    <origin xyz="0 0 0.1" rpy="0 0 0"/> <!-- Mounted 10cm above base_link -->
+  </joint>
+  <!-- Gazebo camera sensor plugin -->
+  <gazebo reference="$(arg uav_name)_camera_link">
+    <sensor type="camera" name="$(arg uav_name)_camera_sensor">
+      <pose>0 0 0 0 0 0</pose>
+      <camera>
+        <horizontal_fov>1.3962634</horizontal_fov>
+        <image>
+          <width>640</width>
+          <height>480</height>
+          <format>R8G8B8</format>
+        </image>
+        <clip>
+          <near>0.05</near>
+          <far>100.0</far>
+        </clip>
+      </camera>
+      <always_on>true</always_on>
+      <update_rate>30.0</update_rate>
+      <visualize>true</visualize>
+      <plugin name="$(arg uav_name)_camera_controller" filename="libgazebo_ros_camera.so">
         <always_on>true</always_on>
         <update_rate>30.0</update_rate>
-        <visualize>true</visualize>
-        <plugin name="${uav_name}_camera_controller" filename="libgazebo_ros_camera.so">
-          <always_on>true</always_on>
-          <update_rate>30.0</update_rate>
-          <camera_name>${uav_name}/camera</camera_name>
-          <image_topic_name>image_raw</image_topic_name>
-          <camera_info_topic_name>camera_info</camera_info_topic_name>
-          <frame_name>${uav_name}_camera_link</frame_name>
-        </plugin>
-      </sensor>
-    </gazebo>
-  </robot>
+        <camera_name>$(arg uav_name)/camera</camera_name>
+        <image_topic_name>image_raw</image_topic_name>
+        <camera_info_topic_name>camera_info</camera_info_topic_name>
+        <frame_name>$(arg uav_name)_camera_link</frame_name>
+      </plugin>
+    </sensor>
+  </gazebo>
 </robot>
